Commit message: Materials namespace troubleshooting finished

File: src/diy_robot_full_cell_description/urdf/cell_model.urdf.xacro (robot description, xacro)
@@ -2,10 +2,14 @@
 <!--this is the main urdf file called while launching and passed to the robot_state_publisher node-->
 <robot xmlns:xacro="http://wiki.ros.org/xacro" name="wer24_robotarm">
-<!-- set robot some gloabal arguments -->
+<!-- set some gloabal arguments (define second order namespaces to avoid name collisions)-->
     <xacro:arg name="name" default="diy_cell"/>
+    <xacro:arg name="tf_prefix" default=""/>
+    <xacro:arg name="tf_prefix_sub" default="sub_"/>
+    <xacro:arg name="tf_prefix_arm" default="arm_"/>
+    <xacro:arg name="tf_prefix_grip" default="grip_"/>
     <link name="world" />
 <!-- import and setup the subframe-->
     <xacro:include filename="$(find diy_robot_full_cell_description)/urdf/subframe_macro.urdf.xacro"/>
-    <xacro:simple_subframe tf_prefix="(arg tf_prefix)" parent="world">
+    <xacro:simple_subframe tf_prefix="$(arg tf_prefix)$(arg tf_prefix_sub)" parent="world">
         <origin xyz="0 0 0" rpy="0 0 0"/>
     </xacro:simple_subframe>
@@ -13,5 +17,4 @@
     <xacro:include filename="$(find diy_robotarm_wer24_description)/urdf/diy_robotarm_macro.urdf.xacro"/>
     <!-- set parameters defined in diy_robotarm_macro.xacro -->
-    <xacro:arg name="tf_prefix" default=""/>
     <xacro:arg name="joint_limit_params" default="$(find diy_robot_full_cell_description)/config/joint_limits.yaml"/>
     <xacro:arg name="kinematics_params" default="$(find diy_robotarm_wer24_description)/config/default_kinematics.yaml"/>
@@ -26,6 +29,6 @@
     <xacro:diy_robotarm
         name="$(arg name)"
-        tf_prefix="$(arg tf_prefix)"
-        parent="$(arg tf_prefix)subframe_link"
+        tf_prefix="$(arg tf_prefix)$(arg tf_prefix_arm)"
+        parent="$(arg tf_prefix)$(arg tf_prefix_sub)subframe_link"
         joint_limits_parameters_file="$(arg joint_limit_params)"
         kinematics_parameters_file="$(arg kinematics_params)"
@@ -38,5 +41,5 @@
 <!-- import and setup the gripper-->
     <xacro:include filename="$(find diy_soft_gripper_description)/urdf/diy_gripper_macro.urdf.xacro"/>
-    <xacro:diy_soft_gripper tf_prefix="(arg tf_prefix)" parent="(arg tf_prefix)link_6">
+    <xacro:diy_soft_gripper tf_prefix="$(arg tf_prefix)$(arg tf_prefix_grip)" parent="$(arg tf_prefix)$(arg tf_prefix_arm)link_6">
         <origin xyz="0 0 0" rpy="0 0 0"/>
     </xacro:diy_soft_gripper>

File: src/diy_robot_full_cell_description/urdf/materials.urdf.xacro (robot description, xacro)
@@ -4,31 +4,33 @@
 https://github.com/ros-simulation/gazebo_ros_demos/blob/kinetic-devel/rrbot_description/urdf/materials.xacro
 -->
-<robot>
-  <material name="black">
-    <color rgba="0.0 0.0 0.0 1.0"/>
-  </material>
-  <material name="blue">
-    <color rgba="0.0 0.0 0.8 1.0"/>
-  </material>
-  <material name="green">
-    <color rgba="0.0 0.8 0.0 1.0"/>
-  </material>
-  <material name="yellow">
-    <color rgba="1.0 1.0 0.0 1.0"/>
-  </material>
-  <material name="grey">
-    <color rgba="0.6 0.6 0.6 1.0"/>
-  </material>
-  <material name="orange">
-    <color rgba="${255/255} ${108/255} ${10/255} 1.0"/>
-  </material>
-  <material name="brown">
-    <color rgba="${222/255} ${207/255} ${195/255} 1.0"/>
-  </material>
-  <material name="red">
-    <color rgba="0.8 0.0 0.0 1.0"/>
-  </material>
-  <material name="white">
-    <color rgba="1.0 1.0 1.0 1.0"/>
-  </material>
+<robot xmlns:xacro="http://wiki.ros.org/xacro">
+  <xacro:macro name="materials" params="tf_prefix">
+    <material name="${tf_prefix}black">
+      <color rgba="0.0 0.0 0.0 1.0"/>
+    </material>
+    <material name="${tf_prefix}blue">
+      <color rgba="0.0 0.0 0.8 1.0"/>
+    </material>
+    <material name="${tf_prefix}green">
+      <color rgba="0.0 0.8 0.0 1.0"/>
+    </material>
+    <material name="${tf_prefix}yellow">
+      <color rgba="1.0 1.0 0.0 1.0"/>
+    </material>
+    <material name="${tf_prefix}grey">
+      <color rgba="0.6 0.6 0.6 1.0"/>
+    </material>
+    <material name="${tf_prefix}orange">
+      <color rgba="${255/255} ${108/255} ${10/255} 1.0"/>
+    </material>
+    <material name="${tf_prefix}brown">
+      <color rgba="${222/255} ${207/255} ${195/255} 1.0"/>
+    </material>
+    <material name="${tf_prefix}red">
+      <color rgba="0.8 0.0 0.0 1.0"/>
+    </material>
+    <material name="${tf_prefix}white">
+      <color rgba="1.0 1.0 1.0 1.0"/>
+    </material>
+  </xacro:macro>
 </robot>

File: src/diy_robot_full_cell_description/urdf/subframe_macro.urdf.xacro (robot description, xacro)
@@ -5,5 +5,5 @@
 <robot xmlns:xacro="http://wiki.ros.org/xacro">
 <!--include materials macro-->
-    <xacro:include filename="$(find diy_robot_full_cell_description)/urdf/materials.urdf.xacro"/>
+   <xacro:include filename="$(find diy_robot_full_cell_description)/urdf/materials.urdf.xacro"/>
 <!--specify parametes for building the simple_subframe (in m)-->
     <xacro:property name="disc_height" value="0.05"/>
@@ -11,4 +11,5 @@
 <!--call this macro in the main urdf.xacro to use a siple desk subframe-->
     <xacro:macro name="simple_subframe" params="tf_prefix parent *origin">
+       <xacro:materials tf_prefix="${tf_prefix}"/>
         <joint name="${tf_prefix}parentTOsubframe" type="fixed">
             <xacro:insert_block name="origin"/>
@@ -18,9 +19,9 @@
         <link name="${tf_prefix}subframe_link">
             <visual>
-                <origin xyz="0 0 ${disc_height/2}" rpy="0 0 0"/>    <!--set the origin to the bottom of the subframe = world -->
+                <origin xyz="0 0 ${-disc_height/2}" rpy="0 0 0"/>    <!--set the origin to the bottom of the subframe = world -->
                 <geometry>
                     <cylinder length="${disc_height/2}" radius="${disc_radius}"/>
                 </geometry>
-                <material name="blue"/>
+                <material name="${tf_prefix}blue"/>
             </visual>
             <collision>
@@ -45,5 +46,5 @@
                     <mesh filename="package://diy_robot_full_cell_description/meshes/visual/subframe.stl" scale="0.001 0.001 0.001"/>
                 </geometry>
-                <material name="black"/>
+                <material name="${tf_prefix}black"/>
             </visual>
             <collision>

Commit message: development finished

File: src/diy_robot_full_cell_description/urdf/cell_model.urdf.xacro (robot description, xacro)
@@ -44,3 +44,10 @@
         <origin xyz="0 0 0" rpy="0 0 0"/>
     </xacro:diy_soft_gripper>
+<!--add a TCP Link for convenience, show TCP reference set in rviz-->
+    <joint name="tcp_joint" type="fixed">
+        <origin xyz="0 0 0.08" rpy="0 0 0"/>
+        <parent link="$(arg tf_prefix)$(arg tf_prefix_grip)base_link"/>
+        <child link="$(arg tf_prefix)tcp_link"/>
+    </joint>
+    <link name="$(arg tf_prefix)tcp_link"/>
 </robot>
