Commit message: remove tcp definition from cell description -> now in gripper description

File: urdf/cell_model.urdf.xacro (robot description, xacro)
@@ -46,10 +46,3 @@
         <origin xyz="0 0 0" rpy="0 0 0"/>
     </xacro:diy_soft_gripper>
-<!--add a TCP Link for convenience, show TCP reference set in rviz-->
-    <joint name="tcp_joint" type="fixed">
-        <origin xyz="0 0 0.08" rpy="0 0 0"/>
-        <parent link="$(arg tf_prefix)$(arg tf_prefix_grip)base_link"/>
-        <child link="$(arg tf_prefix)tcp_link"/>
-    </joint>
-    <link name="$(arg tf_prefix)tcp_link"/>
 </robot>
