Commit message: relocated subframe collision mesh

File: urdf/subframe_macro.urdf.xacro (robot description, xacro)
@@ -26,5 +26,5 @@
             </visual>
             <collision>
-                <origin xyz="0 0 ${disc_height/2}" rpy="0 0 0"/>
+                <origin xyz="0 0 ${-disc_height/2}" rpy="0 0 0"/>
                 <geometry>
                     <cylinder length="${disc_height/2}" radius="${disc_radius}"/>
